Commit message: demo1

File: disarm_ws/src/disarm_simulation/urdf/chaser.xacro (robot description, xacro)
@@ -6,6 +6,6 @@
 <gazebo reference="chaser_body">
     <material>Gazebo/DarkGrey</material>
-    <mu1>0.2</mu1>
-    <mu2>0.2</mu2>
+    <mu1>0</mu1>
+    <mu2>0</mu2>
 </gazebo>
 <link name="chaser_body">
@@ -25,3 +25,6 @@
     </inertial>
 </link>
+  <gazebo>
+  	<plugin name="plannar_mover_plugin" filename="libplannar_mover_plugin.so"> </plugin>
+  </gazebo>
 </robot>

File: disarm_ws/src/disarm_simulation/urdf/disarm.xacro (robot description, xacro)
@@ -83,13 +83,13 @@
   </link>
   <joint
-    name="TopPlate"
+    name="TopFixedPlate"
     type="fixed">
     <origin
-      xyz="0 0 0.27734"
+      xyz="0 0 0"
       rpy="0 0 0" />
     <parent
-      link="Base" />
-    <child
-      link="TopPlate" />
+      link="InnerGuidingRods" />
+    <child
+      link="TopPlate"/>
     <axis
       xyz="0 0 0" />
@@ -136,5 +136,5 @@
   </link>
   <joint
-    name="LeadScrew"
+    name="LeadScrewJoint"
     type="fixed">
     <origin
@@ -149,5 +149,5 @@
   </joint>
   <link
-    name="Actuators">
+    name="Prongs">
     <inertial>
       <origin
@@ -189,18 +189,18 @@
   </link>
   <joint
-    name="Actuators"
+    name="ProngJoint"
     type="fixed">
     <origin
-      xyz="-0.04053 -0.033295 0.27734"
+      xyz="-0.04053 -0.033295 0"
       rpy="0 0 0.087041" />
     <parent
-      link="Base" />
-    <child
-      link="Actuators" />
+      link="TopPlate" />
+    <child
+      link="Prongs" />
     <axis
       xyz="0 0 0" />
   </joint>
   <link
-    name="Sensors">
+    name="InnerGuidingRods">
     <inertial>
       <origin
@@ -242,6 +242,6 @@
   </link>
   <joint
-    name="Sensors"
-    type="fixed">
+    name="innerGRJoint"
+    type="prismatic">
     <origin
       xyz="0 0 0.27734"
@@ -250,8 +250,20 @@
       link="Base" />
     <child
-      link="Sensors" />
-    <axis
-      xyz="0 0 0" />
-  </joint>
+      link="InnerGuidingRods"/>
+    <axis
+      xyz="0 0 1" />
+      <limit lower ="-0.1" upper="0" effort="1000" velocity = "0.2"/>
+      <friction>0.05</friction>
+  </joint>
+   <transmission name="lift_transmission">
+   	<type>transmission_interface/SimpleTransmission</type>
+   	<joint name="innerGRJoint">
+   		<hardwareInterface>hardware_interface/VelocityJointInterface</hardwareInterface>
+   	</joint>
+   	<actuator name="lift_motor">
+      		<hardwareInterface>hardware_interface/VelocityJointInterface</hardwareInterface>
+      		<mechanicalReduction>1</mechanicalReduction>
+    	</actuator>
+    </transmission>
   <link
     name="GuidingRods">
@@ -295,5 +307,5 @@
   </link>
   <joint
-    name="GuidingRods"
+    name="GuidingRodsJoint"
     type="fixed">
     <origin
@@ -303,5 +315,5 @@
       link="Base" />
     <child
-      link="GuidingRods" />
+      link="GuidingRods"/>
     <axis
       xyz="0 0 0" />
@@ -348,15 +360,17 @@
   </link>
   <joint
-    name="Spring"
-    type="fixed">
-    <origin
-      xyz="0 0 0.17416"
+    name="SpringJoint"
+    type="prismatic">
+    <origin
+      xyz="0 0 -0.105"
       rpy="0 0 1.6634" />
     <parent
-      link="Base" />
+      link="TopPlate" />
     <child
       link="Spring" />
     <axis
-      xyz="0 0 0" />
+      xyz="0 0 1" />
+      <limit lower ="0" upper="0" effort="1000" velocity = "0.2"/>
+      <dynamics spring_stiffness="2500" spring_reference="0.06" damping="20.0"/>
   </joint>
   <link
@@ -401,11 +415,11 @@
   </link>
   <joint
-    name="OuterShaft"
+    name="OuterShaftJoint"
     type="fixed">
     <origin
-      xyz="0 0 0.174160571111755"
+      xyz="0 0 -0.105"
       rpy="0 0 1.66344608700645" />
     <parent
-      link="Base" />
+      link="TopPlate" />
     <child
       link="OuterShaft" />
@@ -414,5 +428,5 @@
   </joint>
   <joint name="lidarGlue" type="fixed">
-    <parent link="Sensors"/>
+    <parent link="TopPlate"/>
     <child link="laz_base"/>
     <origin
@@ -427,8 +441,6 @@
     rpy="0 0 0" />
   </joint>
-   <gazebo>
+  <gazebo>
   	<plugin name="disarm_plugin" filename="libdisarm_plugin.so"> </plugin>
-  	<plugin name="mysensor_plugin" filename="libmysensor_plugin.so">
-  	</plugin>
   </gazebo>
 </robot>

File: disarm_ws/src/disarm_simulation/urdf/lidar.xacro (robot description, xacro)
@@ -43,5 +43,5 @@
          <scan>
            <horizontal>
-             <samples>40</samples>
+             <samples>720</samples>
              <resolution>0.25</resolution>
              <min_angle>-${pi/8}</min_angle>
@@ -61,5 +61,4 @@
          </range>
       </ray>
-     <plugin name="mysensor_plugin" filename="libmysensor_plugin.so"> </plugin>
    </sensor>
   </gazebo>
@@ -87,3 +86,6 @@
     <dynamics friction="0.1"/>
   </joint>
+  <gazebo>
+       <plugin name="mysensor_plugin" filename="libmysensor_plugin.so"> </plugin>
+  </gazebo>
 </robot>
